File: headamp/headamp.kicad_sch (KiCad schematic)
At the start: 91 parts, among them J1 MAINS 230V, J401 IN L (RCA), J402 IN R (RCA), J403 jack 6,3mm TRS (DT 770 M 80R), K1 9V, SW1 ON/OFF, SW2 S2 wokal, SW202 S2 wokal (P), SW401 S1 crossfeed, T1 OPT SE 5k:80R (>=25H, 45mA), T201 OPT SE 5k:80R (>=25H, 45mA), T301 EI84 100VA: 230V : 250V/0,15A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, U1 ECC82, U2 EL84 (trioda), U202 EL84 (trioda), U301 LD1085 (LDO)

Commit message: headamp: ELEV/V_RAW drutami, ground breaker wpiety bezposrednio, minimum PWR_FLAG, PDF w ref/
DECYZJA 2026-09-08: na schemacie zostaja tylko symbole GND. ELEV i V_RAW
zamienione z etykiet na realne druty (dzielnik elewacji -> K1.A2 -> minus
zarzenia; K1.A1 -> wezel mostka Schottky zarzenia). Usuniete symbole
Earth_Protective - PE polaczone drutem wprost J1.3 -> ground breaker.
PWR_FLAG zredukowane do 3, kazdy sprawdzony empirycznie (usuniecie
pojedynczo dawalo blad ERC power_pin_not_driven). check.py bez zmian
(asercje juz operowaly na parach pinow z netlisty). ERC 0/0, PDF
eksportowany do headamp/ref/headamp.pdf.

Co-Authored-By: Claude Sonnet 5 <noreply@anthropic.com>
Connections:
- net ELEV is gone; now on net GND: C304.1, C305.2, C306.2, C307.2, C308.2, D305.2 (A), D308.2 (A), D309.2 (A), K1.A2, R304.2, R305.1, R308.2, U1.9 (F2), U2.5 (F2), U202.5 (F2)
- net Earth_Protective: no longer names the net of C309.2, D310.2 (A), D311.1 (K), J1.3 (Pin_3), R309.2
- net V_RAW: no longer names the net of C305.1, C306.1, D305.1 (K), D306.1 (K), D307.1 (K), K1.A1, U301.3 (VI)
Changed lines of the file:
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@@
   (junction (at 77.47 337.82) (diameter 0))
   (junction (at 88.9 337.82) (diameter 0))
-  (junction (at 41.91 326.39) (diameter 0))
   (junction (at 127 313.69) (diameter 0))
   (junction (at 142.24 321.31) (diameter 0))
@@
   (junction (at 384.81 339.09) (diameter 0))
   (junction (at 384.81 361.95) (diameter 0))
+  (junction (at 231.14 330.2) (diameter 0))
+  (junction (at 231.14 297.18) (diameter 0))
   (junction (at 400.05 339.09) (diameter 0))
   (junction (at 405.13 339.09) (diameter 0))
@@
   (wire (pts (xy 40.64 323.85) (xy 41.91 323.85)) (stroke (width 0) (type default)))
   (wire (pts (xy 41.91 323.85) (xy 41.91 326.39)) (stroke (width 0) (type default)))
-  (wire (pts (xy 41.91 326.39) (xy 41.91 335.28)) (stroke (width 0) (type default)))
-  (wire (pts (xy 41.91 326.39) (xy 33.02 326.39)) (stroke (width 0) (type default)))
-  (wire (pts (xy 33.02 326.39) (xy 33.02 328.93)) (stroke (width 0) (type default)))
+  (wire (pts (xy 41.91 326.39) (xy 41.91 355.6)) (stroke (width 0) (type default)))
+  (wire (pts (xy 41.91 355.6) (xy 43.18 355.6)) (stroke (width 0) (type default)))
   (wire (pts (xy 77.47 318.77) (xy 77.47 325.12)) (stroke (width 0) (type default)))
   (wire (pts (xy 77.47 332.74) (xy 77.47 337.82)) (stroke (width 0) (type default)))
@@
   (wire (pts (xy 287.02 361.95) (xy 281.94 361.95)) (stroke (width 0) (type default)))
   (wire (pts (xy 387.35 361.95) (xy 387.35 364.49)) (stroke (width 0) (type default)))
+  (wire (pts (xy 210.82 314.96) (xy 210.82 330.2)) (stroke (width 0) (type default)))
+  (wire (pts (xy 210.82 330.2) (xy 231.14 330.2)) (stroke (width 0) (type default)))
+  (wire (pts (xy 231.14 320.04) (xy 231.14 330.2)) (stroke (width 0) (type default)))
+  (wire (pts (xy 231.14 330.2) (xy 281.94 330.2)) (stroke (width 0) (type default)))
+  (wire (pts (xy 281.94 330.2) (xy 281.94 361.95)) (stroke (width 0) (type default)))
+  (wire (pts (xy 231.14 297.18) (xy 222.25 297.18)) (stroke (width 0) (type default)))
+  (wire (pts (xy 222.25 297.18) (xy 222.25 334.01)) (stroke (width 0) (type default)))
+  (wire (pts (xy 222.25 334.01) (xy 317.5 334.01)) (stroke (width 0) (type default)))
+  (wire (pts (xy 317.5 334.01) (xy 317.5 339.09)) (stroke (width 0) (type default)))
   (wire (pts (xy 400.05 350.52) (xy 400.05 339.09)) (stroke (width 0) (type default)))
   (wire (pts (xy 405.13 350.52) (xy 405.13 339.09)) (stroke (width 0) (type default)))
@@
   (rectangle (start 122 290.47) (end 262 380.47) (stroke (width 0.254) (type default)) (fill (type none)))
   (rectangle (start 262 290.47) (end 495.3 380.47) (stroke (width 0.254) (type default)) (fill (type none)))
-  (label "ELEV" (at 213.36 314.96 0) (effects (font (size 1.27 1.27)) (justify left bottom)))
-  (label "V_RAW" (at 231.14 297.18 0) (effects (font (size 1.27 1.27)) (justify right bottom)))
-  (label "ELEV" (at 231.14 320.04 0) (effects (font (size 1.27 1.27)) (justify right bottom)))
-  (label "V_RAW" (at 320.04 339.09 0) (effects (font (size 1.27 1.27)) (justify left bottom)))
-  (label "ELEV" (at 281.94 361.95 0) (effects (font (size 1.27 1.27)) (justify right bottom)))
   (text "S1 crossfeed: ON = przesluch -14 dB w basie (<700 Hz), OFF = tor prosty" (at 92 20 0) (effects (font (size 1.27 1.27)) (justify left bottom)))
   (text "PE -> wlasna sruba M4 na chassis" (at 22.86 340.36 0) (effects (font (size 1.27 1.27)) (justify left bottom)))
@@
     (instances (project "headamp" (path "/fd162765-1b28-469c-8099-083c76e823f0" (reference "T301") (unit 1))))
   )
-  (symbol (lib_id "power:Earth_Protective") (at 41.91 335.28 0) (unit 1)
-    (in_bom yes) (on_board yes) (dnp no)
-    (property "Reference" "#PE87" (at 41.91 335.28 0) (effects (font (size 1.27 1.27)) hide))
-    (property "Value" "Earth_Protective" (at 41.91 331.47 0) (effects (font (size 1.27 1.27))))
-    (property "Footprint" "" (at 41.91 335.28 0) (effects (font (size 1.27 1.27)) hide))
-    (property "Datasheet" "" (at 41.91 335.28 0) (effects (font (size 1.27 1.27)) hide))
-    (pin "1")
-    (instances (project "headamp" (path "/fd162765-1b28-469c-8099-083c76e823f0" (reference "#PE87") (unit 1))))
-  )
-  (symbol (lib_id "power:PWR_FLAG") (at 33.02 328.93 0) (unit 1)
-    (in_bom yes) (on_board yes) (dnp no)
-    (property "Reference" "#FLG88" (at 33.02 328.93 0) (effects (font (size 1.27 1.27)) hide))
-    (property "Value" "PWR_FLAG" (at 33.02 325.12 0) (effects (font (size 1.27 1.27))))
-    (property "Footprint" "" (at 33.02 328.93 0) (effects (font (size 1.27 1.27)) hide))
-    (property "Datasheet" "" (at 33.02 328.93 0) (effects (font (size 1.27 1.27)) hide))
-    (pin "1")
-    (instances (project "headamp" (path "/fd162765-1b28-469c-8099-083c76e823f0" (reference "#FLG88") (unit 1))))
-  )
   (symbol (lib_id "Device:Varistor") (at 77.47 328.93 0) (unit 1)
     (in_bom yes) (on_board yes) (dnp no)
@@
   (symbol (lib_id "power:GND") (at 160.02 340.36 0) (unit 1)
     (in_bom yes) (on_board yes) (dnp no)
-    (property "Reference" "#GND102" (at 160.02 340.36 0) (effects (font (size 1.27 1.27)) hide))
+    (property "Reference" "#GND100" (at 160.02 340.36 0) (effects (font (size 1.27 1.27)) hide))
     (property "Value" "GND" (at 160.02 344.17 0) (effects (font (size 1.27 1.27))))
     (property "Footprint" "" (at 160.02 340.36 0) (effects (font (size 1.27 1.27)) hide))
     (property "Datasheet" "" (at 160.02 340.36 0) (effects (font (size 1.27 1.27)) hide))
     (pin "1")
-    (instances (project "headamp" (path "/fd162765-1b28-469c-8099-083c76e823f0" (reference "#GND102") (unit 1))))
+    (instances (project "headamp" (path "/fd162765-1b28-469c-8099-083c76e823f0" (reference "#GND100") (unit 1))))
   )
   (symbol (lib_id "Device:R") (at 210.82 308.61 0) (unit 1)
@@
   (symbol (lib_id "power:PWR_FLAG") (at 231.14 294.64 0) (unit 1)
     (in_bom yes) (on_board yes) (dnp no)
-    (property "Reference" "#FLG109" (at 231.14 294.64 0) (effects (font (size 1.27 1.27)) hide))
+    (property "Reference" "#FLG107" (at 231.14 294.64 0) (effects (font (size 1.27 1.27)) hide))
     (property "Value" "PWR_FLAG" (at 231.14 290.83 0) (effects (font (size 1.27 1.27))))
     (property "Footprint" "" (at 231.14 294.64 0) (effects (font (size 1.27 1.27)) hide))
     (property "Datasheet" "" (at 231.14 294.64 0) (effects (font (size 1.27 1.27)) hide))
     (pin "1")
-    (instances (project "headamp" (path "/fd162765-1b28-469c-8099-083c76e823f0" (reference "#FLG109") (unit 1))))
+    (instances (project "headamp" (path "/fd162765-1b28-469c-8099-083c76e823f0" (reference "#FLG107") (unit 1))))
   )
   (symbol (lib_id "power:GND") (at 247.65 327.66 0) (unit 1)
     (in_bom yes) (on_board yes) (dnp no)
-    (property "Reference" "#GND110" (at 247.65 327.66 0) (effects (font (size 1.27 1.27)) hide))
+    (property "Reference" "#GND108" (at 247.65 327.66 0) (effects (font (size 1.27 1.27)) hide))
     (property "Value" "GND" (at 247.65 331.47 0) (effects (font (size 1.27 1.27))))
     (property "Footprint" "" (at 247.65 327.66 0) (effects (font (size 1.27 1.27)) hide))
     (property "Datasheet" "" (at 247.65 327.66 0) (effects (font (size 1.27 1.27)) hide))
     (pin "1")
-    (instances (project "headamp" (path "/fd162765-1b28-469c-8099-083c76e823f0" (reference "#GND110") (unit 1))))
+    (instances (project "headamp" (path "/fd162765-1b28-469c-8099-083c76e823f0" (reference "#GND108") (unit 1))))
   )
   (symbol (lib_id "Device:D") (at 287.02 342.9 270) (unit 1)
@@
   (symbol (lib_id "power:PWR_FLAG") (at 387.35 364.49 180) (unit 1)
     (in_bom yes) (on_board yes) (dnp no)
-    (property "Reference" "#FLG122" (at 387.35 364.49 0) (effects (font (size 1.27 1.27)) hide))
+    (property "Reference" "#FLG120" (at 387.35 364.49 0) (effects (font (size 1.27 1.27)) hide))
     (property "Value" "PWR_FLAG" (at 387.35 368.3 0) (effects (font (size 1.27 1.27))))
     (property "Footprint" "" (at 387.35 364.49 0) (effects (font (size 1.27 1.27)) hide))
     (property "Datasheet" "" (at 387.35 364.49 0) (effects (font (size 1.27 1.27)) hide))
     (pin "1")
-    (instances (project "headamp" (path "/fd162765-1b28-469c-8099-083c76e823f0" (reference "#FLG122") (unit 1))))
+    (instances (project "headamp" (path "/fd162765-1b28-469c-8099-083c76e823f0" (reference "#FLG120") (unit 1))))
   )
   (symbol (lib_id "Valve:ECC81") (at 402.59 339.09 0) (unit 3)
@@
   (symbol (lib_id "power:GND") (at 40.64 347.98 0) (unit 1)
     (in_bom yes) (on_board yes) (dnp no)
-    (property "Reference" "#GND130" (at 40.64 347.98 0) (effects (font (size 1.27 1.27)) hide))
+    (property "Reference" "#GND128" (at 40.64 347.98 0) (effects (font (size 1.27 1.27)) hide))
     (property "Value" "GND" (at 40.64 351.79 0) (effects (font (size 1.27 1.27))))
     (property "Footprint" "" (at 40.64 347.98 0) (effects (font (size 1.27 1.27)) hide))
     (property "Datasheet" "" (at 40.64 347.98 0) (effects (font (size 1.27 1.27)) hide))
     (pin "1")
-    (instances (project "headamp" (path "/fd162765-1b28-469c-8099-083c76e823f0" (reference "#GND130") (unit 1))))
-  )
-  (symbol (lib_id "power:Earth_Protective") (at 43.18 355.6 180) (unit 1)
-    (in_bom yes) (on_board yes) (dnp no)
-    (property "Reference" "#PE131" (at 43.18 355.6 0) (effects (font (size 1.27 1.27)) hide))
-    (property "Value" "Earth_Protective" (at 43.18 359.41 0) (effects (font (size 1.27 1.27))))
-    (property "Footprint" "" (at 43.18 355.6 0) (effects (font (size 1.27 1.27)) hide))
-    (property "Datasheet" "" (at 43.18 355.6 0) (effects (font (size 1.27 1.27)) hide))
-    (pin "1")
-    (instances (project "headamp" (path "/fd162765-1b28-469c-8099-083c76e823f0" (reference "#PE131") (unit 1))))
+    (instances (project "headamp" (path "/fd162765-1b28-469c-8099-083c76e823f0" (reference "#GND128") (unit 1))))
   )
   (sheet_instances (path "/" (page "1")))
