File: headamp/kicad/headamp.kicad_sch (KiCad schematic)
At the start: 91 parts, among them J1 MAINS 230V, J401 IN L (RCA), J402 IN R (RCA), J403 jack 6,3mm TRS (DT 770 M 80R), K1 9V, SW1 ON/OFF, SW2 S2 wokal, SW202 S2 wokal (P), SW401 S1 crossfeed, T1 OPT SE 5k:80R (>=25H, 45mA), T201 OPT SE 5k:80R (>=25H, 45mA), T301 EI84 100VA: 230V : 250V/0,15A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, U1 ECC82, U2 EL84 (trioda), U202 EL84 (trioda), U301 LD1085 (LDO)

Commit message: headamp: WIP - reczne porzadki schematu, K1 podlaczony (V_RAW/ELEV), PWR_FLAG; stan i nastepne kroki w CLAUDE.md
Netlista poprawna (58 sieci). ERC: 3 bledy + 14 ostrzezen z przenumerowania
kanalu P przez KiCad (U3->U1 unit B, zarnik U202B->U4, nadmiarowy PWR_FLAG na
GND, RV2/SW402 jako unit B) - lista do zrobienia w CLAUDE.md "STAN WIP".

Co-Authored-By: Claude Fable 5.1 <noreply@anthropic.com>
Parts:
- removed C201, C403: 220n, symbol Device:C
- removed C202: 1u/25V, symbol Device:C_Polarized
- removed C203: 100u/25V, symbol Device:C_Polarized
- removed C204: 47u/350V, symbol Device:C_Polarized
- removed C205: 100n/400V, symbol Device:C
- removed C206: 470u/25V, symbol Device:C_Polarized
- removed C402: 470n, symbol Device:C
- removed R201, R206: 470k, symbol Device:R
- removed R202, R207, R402: 1k, symbol Device:R
- removed R203: 1k5, symbol Device:R
- removed R204: 47k/2W, symbol Device:R
- removed R205: 10k/2W, symbol Device:R
- removed R208: 270/5W, symbol Device:R
- removed R209: 100, symbol Device:R
- removed R403: 2k2, symbol Device:R
- removed R405: 3k3, symbol Device:R
- removed unit 2 of RV1
- removed SW202: S2 wokal (P), symbol Switch:SW_SPST
- removed unit 1 of SW401
- removed T201: OPT SE 5k:80R (>=25H, 45mA), symbol Device:Transformer_1P_1S
- removed unit 2 of U1
- removed unit 1 of U202
- added C10: 100u/25V, symbol Device:C_Polarized
- added C11: 100n/400V, symbol Device:C
- added C12: 470u/25V, symbol Device:C_Polarized
- added C405, C7: 220n, symbol Device:C
- added C406: 470n, symbol Device:C
- added C8: 47u/350V, symbol Device:C_Polarized
- added C9: 1u/25V, symbol Device:C_Polarized
- added R10, R15: 470k, symbol Device:R
- added R11, R16, R408: 1k, symbol Device:R
- added R12: 1k5, symbol Device:R
- added R13: 47k/2W, symbol Device:R
- added R14: 10k/2W, symbol Device:R
- added R17: 270/5W, symbol Device:R
- added R18: 100, symbol Device:R
- added R407: 2k2, symbol Device:R
- added R409: 3k3, symbol Device:R
- added RV2: 50k log (podwojny), symbol Device:R_Potentiometer_Dual_Separate
- added SW3: S2 wokal, symbol Switch:SW_SPST
- added SW402: S1 crossfeed, symbol Switch:SW_DPDT_x2
- added T2: OPT SE 5k:80R (>=25H, 45mA), symbol Device:Transformer_1P_1S
- added U3: ECC82, symbol Valve:ECC81
- added U4: EL84 (trioda), symbol Valve:EL84
Connections:
- net GND: now also C309.2, C404.1, D310.2 (A), D311.1 (K), R309.2, C10.2, C12.2, C405.1, C8.2, C9.2, R10.2, R12.2, R15.2, R17.2, RV2.3, T2.3 (SA); no longer C309.1, C404.2, D310.1 (K), D311.2 (A), R309.1
- net at C304.1, C305.2, C306.2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: now also C308.1; no longer C308.2
- net at C303.1, K1.12, L1.2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: now also R14.2, T2.1 (AA)
- net at J403.R: now also T2.4 (SB)
- net at R307.1, U1.4 (F1), U1.5 (F1)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: now also C308.2; no longer C308.1
- net at R404.2, R406.1: now also C404.2; no longer C404.1
- net at C401.1, J401.1 (In), R401.1: now also R407.1
- net at J402.1 (In), R404.1: now also C406.1, R408.1
- new net: R16.2, U4.2 (G1)
- new net: C12.1, R17.1, U4.3 (K_G3)
- new net: R18.1, T2.2 (AB), U4.7 (A)
- new net: R18.2, U4.9 (G2)
- new net: C11.1, R13.2, U3.6 (A)
- new net: R11.2, U3.7 (G)
- new net: C9.1, R12.1, SW3.1 (A), U3.8 (K)
- new net: C309.1, D310.1 (K), D311.2 (A), J1.3 (Pin_3), R309.1
- new net: C406.2, R408.2, RV2.1, SW402.5 (B)
- new net: C7.1, RV2.2
- new net: C405.2, R407.2, R409.1
- new net: C8.1, R13.1, R14.1
- new net: C7.2, R10.1, R11.1
- new net: C11.2, R15.1, R16.1
- new net: R409.2, SW402.4 (A)
- new net: C10.1, SW3.2 (B)
Other:
- moved on the sheet: C1, C2, C3, C301, C302, C303, C304, C305, C306, C307, C308, C309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
